File: display_bus_receiver/display_bus_receiver.kicad_sch (KiCad schematic)
At the start: 51 parts, among them U1 74LS245, U10 74LS244, U11 74LS240, U12 74S51, U13 8287, U14 74LS00, U15 74LS08, U16 74LS175, U17 74LS257, U18 74LS374, U19 74LS257, U2 74LS244, U20 74LS244, U21 74LS244, U22 74LS257, U23 8222513, U24 74LS244, U25 74LS273, U26 74LS51, U27 74LS04, U28 74LS27, U29 74LS20, U3 8222512, U30 74LS125, U31 74LS175, U32 74LS244, U33 74LS138, U34 74LS74, U35 74LS00, U36 74LS74, U37 74LS138, U38 74LS74, U39 74LS00, U4 74LS244, U40 74LS20, U41 74LS00, U42 74LS02, U43 74LS373, U44 74LS10, U45 74LS393, U46 74LS51, U47 74LS32, U48 74LS04, U49 74LS20, U5 74LS257, U50 74LS10, U51 74LS32, U6 74LS257, U7 8222511, U8 8287, U9 74LS374

Commit message: Trace 5V and Gnd
Connections:
- net GND: now reaches U30.4
- net GND: now also U1.10 (GND), U10.1 (OEa), U10.10 (GND), U10.19 (OEb), U11.1 (OEa), U11.10 (GND), U11.19 (OEb), U12.7 (GND), U13.10 (GND), U14.7 (GND), U15.7 (GND), U16.8 (GND), U17.8 (GND), U18.10 (GND), U19.8 (GND), U2.10 (GND), U20.10 (GND), U20.15 (I2b), U20.17 (I3b), U21.10 (GND), U22.10 (I1d), U22.13 (I1c), U22.8 (GND), U23.10, U24.10 (GND), U24.13 (I1b), U24.15 (I2b), U24.2 (I0a), U24.4 (I1a), U24.6 (I2a), U24.8 (I3a), U25.10 (GND), U26.7 (GND), U27.7 (GND), U28.7 (GND), U29.7 (GND), U3.10, U30.13, U30.2, U30.7 (GND), U30.9, U31.8 (GND), U32.1 (OEa), U32.10 (GND), U32.19 (OEb), U33.4 (E1), U33.8 (GND), U34.7 (GND), U35.7 (GND), U36.7 (GND), U37.4 (E1), U37.8 (GND), U38.7 (GND), U39.7 (GND), U4.1 (OEa), U4.10 (GND), U4.19 (OEb), U40.7 (GND), U41.7 (GND), U42.7 (GND), U43.1 (OE), U43.10 (GND), U44.7 (GND), U45.7 (GND), U46.7 (GND), U47.7 (GND), U48.7 (GND), U49.7 (GND), U5.10 (I1d), U5.13 (I1c), U5.3 (I1a), U5.6 (I1b), U5.8 (GND), U50.7 (GND), U51.7 (GND), U6.10 (I1d), U6.8 (GND), U7.10, U8.10 (GND), U9.10 (GND)
- net 5V: now reaches U8.20 (VCC)
- net 5V: now also U1.20 (VCC), U10.20 (VCC), U11.20 (VCC), U12.14 (VCC), U13.20 (VCC), U14.14 (VCC), U15.10, U15.12, U15.13, U15.14 (VCC), U15.9, U16.16 (VCC), U17.16 (VCC), U18.20 (VCC), U19.16 (VCC), U2.20 (VCC), U20.20 (VCC), U21.20 (VCC), U22.16 (VCC), U23.20, U24.20 (VCC), U25.20 (VCC), U26.14 (VCC), U27.14 (VCC), U28.14 (VCC), U29.14 (VCC), U3.20, U30.14 (VCC), U31.16 (VCC), U32.20 (VCC), U33.16 (VCC), U34.14 (VCC), U35.14 (VCC), U36.14 (VCC), U37.16 (VCC), U38.14 (VCC), U39.14 (VCC), U4.20 (VCC), U40.10, U40.12, U40.13, U40.14 (VCC), U40.9, U41.10, U41.14 (VCC), U42.14 (VCC), U43.20 (VCC), U44.14 (VCC), U45.14 (VCC), U46.1, U46.10, U46.11, U46.12, U46.13, U46.14 (VCC), U46.9, U47.14 (VCC), U48.14 (VCC), U49.14 (VCC), U5.16 (VCC), U50.14 (VCC), U51.14 (VCC), U6.16 (VCC), U7.20, U9.20 (VCC)
